File: Digital Analog IO/IO.sch (EAGLE design)
At the start: 16 parts, among them IC1 LD117AS33TR

Commit message: update PCB
Parts:
- added JP-PWR-SEL: (no value), pinhead:PINHD-1X3
- added LED-PWR, LED-RSSI: (no value), SparkFun-LED:LED0603
- added PWR-BAT: (no value), pinhead:PINHD-1X2
- added R5, R6: 330R, resistor:R-EU_R0603
- added R7: 3.3K, resistor:R-EU_R0603
- added R8: 1K, resistor:R-EU_R0603
- OPENMOTE: device maxstream:XBEE -> adafruit:XBEE
- R1, R2, R3, R4: device resistor:R-EU_M0805 -> resistor:R-EU_R0603
Connections:
- removed net DIG-IO-2: OPENMOTE.ASSOC/AD5/DIO5, U6.RIGHT
- removed net REG-IN: C1.1, IC1.IN, PWR-SW.S
- new net AN-IN-VCC: OPENMOTE.AD4/DIO4, R7.2, R8.1
- new net ASC: LED-PWR.A, OPENMOTE.ASC/AD5/DIO5
- new net N$1: LED-PWR.C, R5.2
- new net N$2: LED-RSSI.C, R6.2
- new net PWM-1: OPENMOTE.PWM1, U6.RIGHT
- new net RSSI: LED-RSSI.A, OPENMOTE.PWM0/RSSI
- new net V-ADPTR: C2.1, IC1.OUT, JP-PWR-SEL.1
- new net V-BAT: JP-PWR-SEL.3, PWR-BAT.1
- new net V-SEL: JP-PWR-SEL.2, PWR-SW.P
- net 3.3V: now also PWR-SW.S, R7.1; no longer C2.1, IC1.OUT
- net 5V: now also C1.1, IC1.IN; no longer PWR-SW.P
- net AN-IN-0-50MA-1: now also OPENMOTE.AD3/DIO3; no longer OPENMOTE.COORD_SEL/AD3/DIO3
- net DIG-IO-1: now also OPENMOTE.RTS/AD6/DIO6; no longer OPENMOTE.!RTS!/AD6/DIO6
- net GND: now also PWR-BAT.2, R5.1, R6.1, R8.2
Other:
- moved on the sheet: C1, C2, IC1, PWR-ADPTR, PWR-SW, R1, R2, R3, R4, U1, U2, U3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
