File: Mainsnode_v2/Mainsnode_v2/Mainsnode_v2.brd (EAGLE design)
At the start: 160 x 100 mm, 38 parts, among them J2 WIRE_HOLE-14AWG, J3 WIRE_HOLE-14AWG, U1 ATUM, U2 ADE7753, X1 ECS-35-17-5PX-TR

Commit message: Finish schematic, start PCB
Parts:
- removed X1: ECS-35-17-5PX-TR, powercube:CSM-7X
- added C12, C16: C1uF, resistor:C0805
- added C13: C470uF, powercube:CAP_SM_10MM
- added C14, C15: C0.1uF, resistor:C0805
- added C17: C47uF, resistor:C0805
- added D2: DIODE_MMBD914, powercube:SOT-23
- added D3: S1G, powercube:DO-214AC
- added IC1: 7805T, adafruit:TO220H
- added J4, J5, J6, J7: HOLE, powercube:HOLE-0.125
- added K1: S216S01F, powercube:RELAY_SX16S0X
- added L4: MPZ2012S300A, powercube:0805_RESISTOR
- added Q1: STGD5NB120SZT4, powercube:DPAK
- added Q2: 3.579545MHz, crystal:HC49/S
- added R12: R330, resistor:R0805
- added R13: R100K, resistor:R0805
- added R14, R16: R200K, resistor:R0805
- added R15, R17: R510K, resistor:R0805
- added R18: R120K, resistor:R0805
- added R19: R12.4K, resistor:R0805
- added TP1, TP2, TP3, TP_ADE_CF, TP_ADE_CS, TP_ADE_IRQ, TP_ADE_ZX, TP_MISO, TP_MOSI, TP_SCLK: PTR1PAD1-13, testpad:P1-13
- added U$1: FDV301N, powercube:SOT-23
- added U4: SR086SG-G, powercube:SR086
- moved J1 273.8 mm to (64.0, 23.5), turned to 180 degrees
- moved C7 185.1 mm to (31.8, 44.1), turned to 270 degrees
- moved C8 183.5 mm to (17.1, 44.1), turned to 270 degrees
- moved C6 161.3 mm to (31.8, 39.4), turned to 90 degrees
- moved C5 154.7 mm to (29.2, 39.4), turned to 90 degrees
- moved U3 152.1 mm to (15.2, 33.7), turned to 270 degrees
- moved C4 146.0 mm to (30.8, 33.0)
- moved C3 139.6 mm to (32.1, 29.5), turned to 270 degrees
- moved C2 131.6 mm to (27.0, 29.5), turned to 270 degrees
- moved C1 125.3 mm to (24.4, 29.5), turned to 270 degrees
- moved R6 124.8 mm to (29.5, 29.5), turned to 270 degrees
- moved R5 114.9 mm to (21.9, 29.5), turned to 90 degrees
- moved U2 113.6 mm to (23.5, 37.1), turned to 180 degrees
- moved R3 91.3 mm to (34.0, -18.7), turned to 270 degrees
- moved R4 90.7 mm to (31.4, -18.7), turned to 270 degrees
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Connections:
- removed net /ADE_IRQ: U2.14
- removed net N$6: U3.2
- new net ADE_CS: TP_ADE_CS.TP, U1.5, U3.2
- new net ADE_IRQ: TP_ADE_IRQ.TP, U1.6, U2.14
- new net N$11: D2.3, K1.3, R12.1
- new net N$12: D2.1, K1.4, U$1.3
- new net N$13: D3.CATHODE, Q1.P$2, R14.2, R15.2
- new net N$14: R14.1, R16.2
- new net N$15: R15.1, R17.2
- new net N$17: R17.1, U4.1
- new net N$18: Q1.P$1, U4.8
- new net N$21: C15.2, U4.7
- new net N$23: R18.1, R19.2, U4.5
- new net RELAY_CTRL: R13.1, U$1.1, U1.7
- new net VDC: C12.1, C13.+, C15.1, C16.1, IC1.1, Q1.P$3, R18.2, U4.6
- net 3V3: now also C14.1, R13.2, U1.1, U4.4
- net 5V: now also C17.1, IC1.3, R12.2
- net ADE_CF: now also TP_ADE_CF.TP
- net ADE_ZX: now also TP_ADE_ZX.TP
- net GND: now also C12.2, C13.-, C14.2, C16.2, C17.2, IC1.2, L4.P$2, R16.1, R19.1, U$1.2, U1.32, U4.2, U4.3, U4.PAD
- net LOAD_PHASE: now also K1.1
- net MISO: now also TP_MISO.TP
- net MOSI: now also TP_MOSI.TP, U1.20
- net N$19: now also Q2.2; no longer X1.2
- net N$20: now also Q2.1; no longer X1.1
- net SCLK: now also TP_SCLK.TP
- net V1N: now also TP2.TP
- net V1P: now also TP1.TP
- net V2P: now also TP3.TP
- net WALL_NEUTRAL: now also L4.P$1
- net WALL_PHASE: now also D3.ANNODE, K1.2
Other:
- board size 160 x 100 mm -> 72.6 x 47.1 mm
