File: Mainsnode_v2/Mainsnode_v2_wifi/Mainsnode_v2_wifi.sch (EAGLE design)
At the start: 70 parts, among them IC1 7805T, J2 WIRE_HOLE-14AWG, J3 WIRE_HOLE-14AWG, J4 HOLE, J5 HOLE, J6 HOLE, J7 HOLE, K1 S216S01F, Q1 STGD5NB120SZT4, Q2 3.579545MHz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

Commit message: Start route wifi board
Parts:
- removed C5, C6: C1uF, resistor:C-EUC0805
- removed IC1: 7805T, adafruit:7805T
- removed JP1: (no value), pinhead:PINHD-2X4
- removed L2, L3: EMI_SUPRESSION_FERRITE_BEAD, powercube:EMI_SUPRESSION_FERRITE_BEAD
- removed TP_ADE_CF, TP_ADE_CS, TP_ADE_IRQ, TP_ADE_ZX, TP_MISO, TP_MOSI, TP_SCK: PTR1PAD1-13, testpad:PTR1PAD1-13
- added C18, C19: C10uF, resistor:C-EUC0805
- added IC2: LD117AS50TR, v-reg:LD117AS50TR
- added R7: R10K, resistor:R-EU_R0805
- added U$3: ESP8266, tigorcustom:ESP8266
- added U$4, U$5: BLM18BB151SN1, tigorcustom:L0603
- U$1: device SparkFun-Boards:ARDUINO_PRO_MINI -> tigorcustom:ARDUINO_PRO_MINI
Connections:
- net 3V3: now also U$3.VCC; no longer JP1.7
- net 5V: now also C19.1, IC2.OUT, R7.1; no longer C6.1, IC1.VO
- net ADE_CF: now also U$1.*5; no longer TP_ADE_CF.TP, U$1.A3
- net ADE_CS: no longer TP_ADE_CS.TP
- net ADE_IRQ: now also R7.2, U$1.*3; no longer TP_ADE_IRQ.TP, U$1.A1
- net ADE_ZX: now also U$1.4; no longer TP_ADE_ZX.TP, U$1.A2
- net DBG_RXI: now also U$1.A3; no longer U$1.*5
- net DBG_TXO: now also U$1.A2; no longer U$1.4
- net GND: now also C18.2, C19.2, IC2.ADJ, U$3.GND; no longer C5.2, C6.2, IC1.GND, JP1.2
- net LOAD_NEUTRAL: now also U$4.P$1; no longer L2.P$1
- net MISO: no longer TP_MISO.TP
- net MOSI: no longer TP_MOSI.TP
- net N$14: now also U$4.P$2; no longer L2.P$2
- net N$15: now also U$5.P$2; no longer L3.P$2
- net RELAY_CTRL: now also U$1.A1; no longer U$1.*3
- net RXI: now also U$3.TXD; no longer JP1.1
- net SCK: no longer TP_SCK.TP
- net TXO: now also U$3.RXD; no longer JP1.8
- net VDC: now also C18.1, IC2.IN; no longer C5.1, IC1.VI
- net WALL_NEUTRAL: now also U$5.P$1; no longer L3.P$1

Commit message: Finish route wifi board and order component
Parts:
- removed U$2: FDV301N, powercube:FDV301N
- added L2: BLM31PG330SN1, resistor:L-EUL3216C
- added Q3: MMBT2222A, SparkFun-DiscreteSemi:TRANSISTOR_NPNMMBT2222A
- R17: value R100K -> R220
Connections:
- new net N$19: Q3.B, R17.2
- net 3V3: no longer R17.1
- net GND: now also Q3.E; no longer U$2.S
- net N$17: now also L2.2
- net N$18: now also Q3.C; no longer U$2.D
- net RELAY_CTRL: now also R17.1, U$1.*10; no longer R17.2, U$1.A1, U$2.G
- net WALL_PHASE: now also L2.1
Other:
- moved on the sheet: R17
Changed lines of the file:
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@@
 <part name="D3" library="semicon-smd-ipc" deviceset="D-" device="SOD-80" value="1N4148"/>
 <part name="R16" library="resistor" deviceset="R-EU_" device="R0805" value="R220"/>
-<part name="U$2" library="powercube" deviceset="FDV301N" device=""/>
-<part name="R17" library="resistor" deviceset="R-EU_" device="R0805" value="R100K"/>
+<part name="R17" library="resistor" deviceset="R-EU_" device="R0805" value="R220"/>
 <part name="JP2" library="pinhead" deviceset="PINHD-1X4" device=""/>
 <part name="J4" library="powercube" deviceset="HOLE" device=""/>
@@
 <part name="U$4" library="tigorcustom" deviceset="L0603" device="" value="BLM18BB151SN1"/>
 <part name="U$5" library="tigorcustom" deviceset="L0603" device="" value="BLM18BB151SN1"/>
+<part name="L2" library="resistor" deviceset="L-EU" device="L3216C" value="BLM31PG330SN1"/>
+<part name="Q3" library="SparkFun-DiscreteSemi" deviceset="TRANSISTOR_NPN" device="MMBT2222A" value="MMBT2222A"/>
 </parts>
 <sheets>
@@
 <instance part="D3" gate="G$1" x="241.3" y="22.86" rot="R90"/>
 <instance part="R16" gate="G$1" x="256.54" y="35.56" rot="R180"/>
-<instance part="U$2" gate="G$1" x="241.3" y="10.16"/>
-<instance part="R17" gate="G$1" x="233.68" y="20.32" rot="R270"/>
+<instance part="R17" gate="G$1" x="228.6" y="10.16"/>
 <instance part="JP2" gate="A" x="182.88" y="119.38"/>
 <instance part="J4" gate="G$1" x="124.46" y="231.14"/>
@@
 <instance part="U$4" gate="G$1" x="335.28" y="96.52" rot="R90"/>
 <instance part="U$5" gate="G$1" x="335.28" y="73.66" rot="R90"/>
+<instance part="L2" gate="G$1" x="335.28" y="45.72" rot="R90"/>
+<instance part="Q3" gate="G$1" x="238.76" y="10.16"/>
 </instances>
 <busses>
@@
 <wire x1="312.42" y1="53.34" x2="309.88" y2="53.34" width="0.1524" layer="91"/>
 <label x="292.1" y="53.34" size="1.778" layer="95"/>
+<wire x1="325.12" y1="53.34" x2="325.12" y2="45.72" width="0.1524" layer="91"/>
+<pinref part="L2" gate="G$1" pin="1"/>
+<wire x1="325.12" y1="45.72" x2="330.2" y2="45.72" width="0.1524" layer="91"/>
 </segment>
 <segment>
@@
 </segment>
 <segment>
-<pinref part="U$2" gate="G$1" pin="S"/>
-<wire x1="241.3" y1="5.08" x2="241.3" y2="2.54" width="0.1524" layer="91"/>
-<label x="241.3" y="2.54" size="1.778" layer="95"/>
-</segment>
-<segment>
 <pinref part="JP2" gate="A" pin="4"/>
 <wire x1="180.34" y1="116.84" x2="177.8" y2="116.84" width="0.1524" layer="91"/>
@@
 <wire x1="66.04" y1="124.46" x2="66.04" y2="121.92" width="0.1524" layer="91"/>
 <label x="66.04" y="121.92" size="1.778" layer="95"/>
+</segment>
+<segment>
+<pinref part="Q3" gate="G$1" pin="E"/>
+<wire x1="241.3" y1="5.08" x2="241.3" y2="2.54" width="0.1524" layer="91"/>
+<label x="241.3" y="2.54" size="1.778" layer="95"/>
 </segment>
 </net>
@@
 </segment>
 <segment>
-<pinref part="R17" gate="G$1" pin="1"/>
-<wire x1="233.68" y1="25.4" x2="231.14" y2="25.4" width="0.1524" layer="91"/>
-<label x="228.6" y="25.4" size="1.778" layer="95"/>
-</segment>
-<segment>
 <pinref part="JP2" gate="A" pin="1"/>
 <wire x1="180.34" y1="124.46" x2="177.8" y2="124.46" width="0.1524" layer="91"/>
@@
 <pinref part="R14" gate="G$1" pin="1"/>
 <wire x1="345.44" y1="53.34" x2="350.52" y2="53.34" width="0.1524" layer="91"/>
+<pinref part="L2" gate="G$1" pin="2"/>
+<wire x1="340.36" y1="45.72" x2="345.44" y2="45.72" width="0.1524" layer="91"/>
+<wire x1="345.44" y1="45.72" x2="345.44" y2="53.34" width="0.1524" layer="91"/>
 </segment>
 </net>
@@
 <pinref part="D3" gate="G$1" pin="A"/>
 <wire x1="243.84" y1="20.32" x2="241.3" y2="20.32" width="0.1524" layer="91"/>
-<pinref part="U$2" gate="G$1" pin="D"/>
 <wire x1="241.3" y1="15.24" x2="241.3" y2="20.32" width="0.1524" layer="91"/>
+<pinref part="Q3" gate="G$1" pin="C"/>
 </segment>
 </net>
 <net name="RELAY_CTRL" class="0">
 <segment>
-<pinref part="R17" gate="G$1" pin="2"/>
-<wire x1="233.68" y1="15.24" x2="233.68" y2="10.16" width="0.1524" layer="91"/>
-<pinref part="U$2" gate="G$1" pin="G"/>
-<wire x1="233.68" y1="10.16" x2="236.22" y2="10.16" width="0.1524" layer="91"/>
-<wire x1="233.68" y1="10.16" x2="231.14" y2="10.16" width="0.1524" layer="91"/>
-<label x="215.9" y="10.16" size="1.778" layer="95"/>
-</segment>
-<segment>
-<pinref part="U$1" gate="G$1" pin="A1"/>
-<wire x1="228.6" y1="170.18" x2="231.14" y2="170.18" width="0.1524" layer="91"/>
-<label x="231.14" y="170.18" size="1.778" layer="95"/>
+<pinref part="U$1" gate="G$1" pin="*10"/>
+<wire x1="228.6" y1="157.48" x2="231.14" y2="157.48" width="0.1524" layer="91"/>
+<label x="231.14" y="157.48" size="1.778" layer="95"/>
+</segment>
+<segment>
+<pinref part="R17" gate="G$1" pin="1"/>
+<wire x1="223.52" y1="10.16" x2="220.98" y2="10.16" width="0.1524" layer="91"/>
+<label x="208.28" y="10.16" size="1.778" layer="95"/>
 </segment>
 </net>
@@
 </segment>
 </net>
+<net name="N$19" class="0">
+<segment>
+<pinref part="R17" gate="G$1" pin="2"/>
+<pinref part="Q3" gate="G$1" pin="B"/>
+<wire x1="233.68" y1="10.16" x2="236.22" y2="10.16" width="0.1524" layer="91"/>
+</segment>
+</net>
